Commit message: checked lidar measurements using object a known distance away from base link, changed frame id to match driver

File: urdf/red_truck.urdf (robot description, URDF)
Before this commit: robot red_truck, 4 links, 3 joints
Links:
- removed link lidar
- added link laser
Joints:
- removed joint lidar_joint
- added joint laser_joint: type fixed, parent base_link, child laser, origin xyz=0.41 -0.01 0.185 rpy=0 0 3.141592

Commit message: Corrected pi rounding

File: urdf/red_truck.urdf (robot description, URDF)
Before this commit: robot red_truck, 4 links, 3 joints
Joints:
- joint laser_joint: origin xyz=0.41 -0.01 0.185 rpy=0 0 3.141592 -> xyz=0.41 -0.01 0.185 rpy=0 0 3.141593
