Commit message: Rounded pi correctly

File: urdf/blue_truck.urdf (robot description, URDF)
Before this commit: robot red_truck, 4 links, 3 joints
Joints:
- joint lidar_joint: origin xyz=0.447675 0.0 0.143 rpy=0 0 3.141592 -> xyz=0.447675 0.0 0.143 rpy=0 0 3.141593

Commit message: Corrected joint name (lidar->laser)

File: urdf/blue_truck.urdf (robot description, URDF)
Before this commit: robot red_truck, 4 links, 3 joints
Links:
- removed link lidar
- added link laser
Joints:
- removed joint lidar_joint
- added joint laser_joint: type fixed, parent base_link, child laser, origin xyz=0.447675 0.0 0.143 rpy=0 0 3.141593

Commit message: changed footprint to base_footprint

File: urdf/blue_truck.urdf (robot description, URDF)
Before this commit: robot red_truck, 4 links, 3 joints
Links:
- removed link footprint
- added link base_footprint
Joints:
- joint footprint_joint: child footprint -> base_footprint

File: urdf/red_truck.urdf (robot description, URDF)
Before this commit: robot red_truck, 4 links, 3 joints
Links:
- removed link footprint
- added link base_footprint
Joints:
- joint footprint_joint: child footprint -> base_footprint
